File: pcb/controller/vertebra.sch (KiCad schematic (older format))
At the start: 10 parts, among them J1 AC, J2 CONN_02X10, J3 GND, U1 74LS165

Commit message: modified vertebra to match brain
Connections:
- net CLOCK: now also TO_BRAIN1.7 (P7), TO_TAIL1.7 (P7); no longer TO_BRAIN1.6 (P6), TO_TAIL1.6 (P6)
- net GND: now also TO_BRAIN1.3 (P3), TO_TAIL1.3 (P3), U1.15 (CE)
- net SERIAL_IN: now also TO_TAIL1.6 (P6); no longer TO_TAIL1.5 (P5)
- net SERIAL_OUT: now also TO_BRAIN1.6 (P6); no longer TO_BRAIN1.5 (P5)
- net VCC: now also TO_BRAIN1.5 (P5), TO_TAIL1.5 (P5); no longer TO_BRAIN1.3 (P3), TO_TAIL1.3 (P3)
- removed net ENABLE: TO_BRAIN1.7 (P7), TO_TAIL1.7 (P7), U1.15 (CE)
Other:
- moved on the sheet: TO_TAIL1
Changed lines of the file:
@@
 LIBS:zetex
 LIBS:Zilog
-LIBS:spine-cache
 EELAYER 25 0
 EELAYER END
@@
 Text GLabel 3500 4350 0    39   Input ~ 0
 CLOCK
-Text GLabel 3500 4450 0    39   Input ~ 0
-ENABLE
 Text GLabel 2350 3200 1    60   Input ~ 0
 N_ENCODER
@@
 	1    0    0    -1
 $EndComp
-Text GLabel 4300 1050 0    39   Input ~ 0
+Text GLabel 4350 1100 0    39   Input ~ 0
 SERIAL_IN
-Text GLabel 3350 1050 2    39   Input ~ 0
+Text GLabel 3400 1100 2    39   Input ~ 0
 SERIAL_OUT
 $Comp
@@
 	0    -1   -1   0
 $EndComp
-Text GLabel 3850 800  1    39   Input ~ 0
+Text GLabel 3800 800  1    39   Input ~ 0
 N_START
 $Comp
 L GND #PWR015
 U 1 1 59ACC792
-P 3700 800
-F 0 "#PWR015" H 3700 550 50  0001 C CNN
-F 1 "GND" H 3700 650 50  0000 C CNN
-F 2 "" H 3700 800 50  0001 C CNN
-F 3 "" H 3700 800 50  0001 C CNN
-	1    3700 800
+P 3450 800
+F 0 "#PWR015" H 3450 550 50  0001 C CNN
+F 1 "GND" V 3450 600 50  0000 C CNN
+F 2 "" H 3450 800 50  0001 C CNN
+F 3 "" H 3450 800 50  0001 C CNN
+	1    3450 800
 	1    0    0    1
 $EndComp
@@
 	-1   0    0    -1
 $EndComp
-Text GLabel 4150 800  1    39   Input ~ 0
+Text GLabel 4000 800  1    39   Input ~ 0
 CLOCK
-Text GLabel 4050 800  1    39   Input ~ 0
-ENABLE
-Text GLabel 3950 800  1    39   Input ~ 0
+Text GLabel 3900 800  1    39   Input ~ 0
 N_LOAD
 $Comp
 L CONN_02X08 TO_TAIL1
 U 1 1 59ACD5F0
-P 4600 1250
-F 0 "TO_TAIL1" H 4600 1700 50  0000 C CNN
-F 1 "CONN_02X08" V 4600 1250 50  0000 C CNN
-F 2 "Pin_Headers:Pin_Header_Straight_2x08_Pitch2.54mm_SMD" H 4600 50  50  0001 C CNN
-F 3 "" H 4600 50  50  0001 C CNN
-	1    4600 1250
+P 4650 1250
+F 0 "TO_TAIL1" H 4650 1700 50  0000 C CNN
+F 1 "CONN_02X08" V 4650 1250 50  0000 C CNN
+F 2 "Pin_Headers:Pin_Header_Straight_2x08_Pitch2.54mm_SMD" H 4650 50  50  0001 C CNN
+F 3 "" H 4650 50  50  0001 C CNN
+	1    4650 1250
 	-1   0    0    -1
 $EndComp
@@
 P 3350 800
 F 0 "#PWR018" H 3350 650 50  0001 C CNN
-F 1 "+12V" H 3350 950 50  0000 C CNN
+F 1 "+12V" V 3350 1000 50  0000 C CNN
 F 2 "" H 3350 800 50  0001 C CNN
 F 3 "" H 3350 800 50  0001 C CNN
@@
 P 3550 800
 F 0 "#PWR019" H 3550 650 50  0001 C CNN
-F 1 "VCC" H 3550 950 50  0000 C CNN
+F 1 "VCC" V 3550 1000 50  0000 C CNN
 F 2 "" H 3550 800 50  0001 C CNN
 F 3 "" H 3550 800 50  0001 C CNN
@@
 	-1   0    0    -1
 $EndComp
-NoConn ~ 4300 1600
+NoConn ~ 4350 1600
 $Comp
 L CONN_01X01 J1
@@
 $EndComp
 Wire Wire Line
-	4900 1050 4900 1100
-Wire Wire Line
-	4900 1150 4900 1200
-Wire Wire Line
-	4900 1250 4900 1300
-Wire Wire Line
-	4900 1350 4900 1400
-Wire Wire Line
-	4900 1450 4900 1500
-Wire Wire Line
-	4900 1550 4900 1600
-Wire Wire Line
-	4900 1100 4850 1100
-Wire Wire Line
-	4900 1200 4850 1200
-Wire Wire Line
-	4900 1300 4850 1300
-Wire Wire Line
-	4900 1400 4850 1400
-Wire Wire Line
-	4900 1500 4850 1500
-Wire Wire Line
-	4900 1600 4850 1600
+	4950 1050 4950 1100
+Wire Wire Line
+	4950 1150 4950 1200
+Wire Wire Line
+	4950 1250 4950 1300
+Wire Wire Line
+	4950 1350 4950 1400
+Wire Wire Line
+	4950 1450 4950 1500
+Wire Wire Line
+	4950 1550 4950 1600
+Wire Wire Line
+	4950 1100 4900 1100
+Wire Wire Line
+	4950 1200 4900 1200
+Wire Wire Line
+	4950 1300 4900 1300
+Wire Wire Line
+	4950 1400 4900 1400
+Wire Wire Line
+	4950 1500 4900 1500
+Wire Wire Line
+	4950 1600 4900 1600
 Wire Wire Line
 	2750 1050 2750 1100
@@
 	2800 1450 2750 1450
 Wire Wire Line
-	3300 1550 4200 1550
+	3300 1550 4100 1550
 Wire Wire Line
 	2800 1550 2750 1550
@@
 	2750 1350 2750 1400
 Wire Wire Line
-	4250 1550 4900 1550
-Wire Wire Line
-	4150 1450 4900 1450
-Wire Wire Line
-	4050 1350 4900 1350
-Wire Wire Line
-	3950 1250 4900 1250
-Wire Wire Line
-	2750 1300 3950 1300
+	4150 1550 4950 1550
+Wire Wire Line
+	4050 1450 4950 1450
+Wire Wire Line
+	3950 1350 4950 1350
+Wire Wire Line
+	3850 1250 4950 1250
+Wire Wire Line
+	2750 1300 3850 1300
 Wire Wire Line
 	3300 3300 3300 3950
@@
 Connection ~ 3300 2850
 Wire Wire Line
-	2750 1500 4150 1500
-Wire Wire Line
-	3300 1450 4100 1450
-Wire Wire Line
-	3300 1350 4000 1350
-Wire Wire Line
-	2750 1400 4050 1400
-Wire Wire Line
-	4350 1600 4300 1600
-Wire Wire Line
-	4200 1500 4350 1500
-Wire Wire Line
-	4100 1400 4350 1400
-Wire Wire Line
-	4000 1300 4350 1300
-Wire Wire Line
-	3300 950  4900 950
-Wire Wire Line
-	4850 1000 4900 1000
-Wire Wire Line
-	3300 850  4900 850
-Wire Wire Line
-	4850 900  4900 900
+	2750 1500 4050 1500
+Wire Wire Line
+	3300 1450 4000 1450
+Wire Wire Line
+	3300 1350 3900 1350
+Wire Wire Line
+	2750 1400 3950 1400
+Wire Wire Line
+	4400 1600 4350 1600
+Wire Wire Line
+	4100 1500 4400 1500
+Wire Wire Line
+	4000 1400 4400 1400
+Wire Wire Line
+	3900 1300 4400 1300
+Wire Wire Line
+	3300 950  4950 950
+Wire Wire Line
+	4900 1000 4950 1000
+Wire Wire Line
+	3300 850  4950 850
+Wire Wire Line
+	4900 900  4950 900
 Wire Wire Line
 	2750 850  2800 850
@@
 	2750 850  2750 900
 Wire Wire Line
-	4900 1000 4900 950
-Wire Wire Line
-	4900 900  4900 850
-Wire Wire Line
-	2750 1600 4250 1600
+	4950 1000 4950 950
+Wire Wire Line
+	4950 900  4950 850
+Wire Wire Line
+	2750 1600 4150 1600
 Wire Wire Line
 	2750 1550 2750 1600
@@
 Connection ~ 3350 850
 Wire Wire Line
-	2750 1000 4350 1000
-Wire Wire Line
-	3850 800  3850 1250
-Wire Wire Line
-	3950 1300 3950 1250
-Wire Wire Line
-	4000 1350 4000 1300
-Wire Wire Line
-	4050 1400 4050 1350
-Wire Wire Line
-	4100 1450 4100 1400
-Wire Wire Line
-	4150 1500 4150 1450
-Wire Wire Line
-	4200 1550 4200 1500
-Wire Wire Line
-	4250 1600 4250 1550
-Wire Wire Line
-	3850 1250 3300 1250
-Wire Wire Line
-	2750 1200 4350 1200
+	2750 1000 4400 1000
+Wire Wire Line
+	3800 800  3800 1250
+Wire Wire Line
+	3850 1300 3850 1250
+Wire Wire Line
+	3900 1350 3900 1300
+Wire Wire Line
+	3950 1400 3950 1350
+Wire Wire Line
+	4000 1450 4000 1400
+Wire Wire Line
+	4050 1500 4050 1450
+Wire Wire Line
+	4100 1550 4100 1500
+Wire Wire Line
+	4150 1600 4150 1550
+Wire Wire Line
+	3800 1250 3300 1250
+Wire Wire Line
+	2750 1200 4400 1200
 Wire Wire Line
 	2750 1200 2750 1150
@@
 	2750 1150 2800 1150
 Wire Wire Line
-	2750 900  4350 900
-Wire Wire Line
-	4150 800  4150 1100
-Wire Wire Line
-	4050 800  4050 1150
-Connection ~ 4050 1150
-Wire Wire Line
-	3950 800  3950 1200
-Wire Wire Line
-	3700 800  3700 1000
-Connection ~ 3700 1000
-Wire Wire Line
-	3550 800  3550 950
-Connection ~ 3550 950
+	2750 900  4400 900
+Wire Wire Line
+	3900 800  3900 1200
 Connection ~ 3350 900
 Wire Wire Line
-	4300 1050 4900 1050
-Wire Wire Line
-	3300 1050 3350 1050
-Wire Wire Line
-	2750 1100 4350 1100
-Connection ~ 4150 1100
-Wire Wire Line
-	3300 1150 4900 1150
-Connection ~ 3950 1200
+	3300 1050 4950 1050
+Wire Wire Line
+	3300 1150 4950 1150
+Connection ~ 3900 1200
+$Comp
+L GND #PWR020
+U 1 1 59B44E79
+P 3500 4450
+F 0 "#PWR020" H 3500 4200 50  0001 C CNN
+F 1 "GND" V 3500 4250 50  0000 C CNN
+F 2 "" H 3500 4450 50  0001 C CNN
+F 3 "" H 3500 4450 50  0001 C CNN
+	1    3500 4450
+	0    1    -1   0
+$EndComp
+Wire Wire Line
+	3450 800  3450 1000
+Connection ~ 3450 950
+Connection ~ 3450 1000
+Wire Wire Line
+	4000 800  4000 1150
+Connection ~ 4000 1150
+Wire Wire Line
+	4350 1100 4400 1100
+Wire Wire Line
+	2750 1100 3400 1100
+Wire Wire Line
+	3550 800  3550 1050
+Connection ~ 3550 1050
 $EndSCHEMATC
