File: pcb/controller/brain.kicad_pcb (KiCad board)
At the start: 2 copper layers, 0 parts

Commit message: designed v0.1 of brain board
Parts:
- added C1: 1uF, Capacitors_SMD:C_0603_HandSoldering, F.Cu at (32.4, 189.2)
- added C2: 1uF, Capacitors_SMD:C_0603_HandSoldering, F.Cu at (55.9, 188.6)
- added C3: 1uF, Capacitors_SMD:C_0603_HandSoldering, F.Cu at (69.8, 188.6)
- added C4: 1uF, Capacitors_SMD:C_0603_HandSoldering, F.Cu at (83.8, 188.6)
- added C5: 1uF, Capacitors_SMD:C_0603_HandSoldering, F.Cu at (32.4, 185.4)
- added G***: LOGO, LOGO, B.Cu at (80.6, 185.4)
- added G***: LOGO, LOGO, B.Cu at (66.7, 186.1)
- added G***: LOGO, LOGO, B.Cu at (52.7, 186.1)
- added G***: LOGO, LOGO, B.Cu at (28.6, 182.2)
- added G***: LOGO, LOGO, B.Cu at (52.7, 173.4)
- added G***: LOGO, LOGO, B.Cu at (66.7, 173.4)
- added G***: LOGO, LOGO, B.Cu at (80.6, 173.4)
- added GND1: TP, Measurement_Points:Measurement_Point_Round-SMD-Pad_Small, F.Cu at (18.4, 177.2)
- added J1: CONN_02X08, Pin_Headers:Pin_Header_Straight_2x08_Pitch2.54mm_SMD, F.Cu at (34.3, 172.1)
- added J10: break, breakaway:0.35mil_square, F.Cu at (47.0, 193.0)
- added J11: break, breakaway:0.35mil_square, B.Cu at (44.5, 193.0)
- added J12: break, breakaway:0.35mil_square, B.Cu at (47.0, 193.0)
- added J13: break, breakaway:0.35mil_square, F.Cu at (44.5, 194.3)
- added J14: break, breakaway:0.35mil_square, F.Cu at (47.0, 194.3)
- added J15: break, breakaway:0.35mil_square, B.Cu at (44.5, 194.3)
- added J16: break, breakaway:0.35mil_square, B.Cu at (47.0, 194.3)
- added J17: break, breakaway:0.35mil_square, F.Cu at (58.4, 191.8)
- added J18: break, breakaway:0.35mil_square, F.Cu at (61.0, 191.8)
- added J19: break, breakaway:0.35mil_square, B.Cu at (58.4, 191.8)
- added J2: CONN_01X08, Pin_Headers:Pin_Header_Straight_1x08_Pitch2.54mm_SMD_Pin1Right, F.Cu at (50.2, 178.4)
- added J20: break, breakaway:0.35mil_square, B.Cu at (61.0, 191.8)
- added J21: break, breakaway:0.35mil_square, F.Cu at (58.4, 193.0)
- added J22: break, breakaway:0.35mil_square, F.Cu at (61.0, 193.0)
- added J23: break, breakaway:0.35mil_square, B.Cu at (58.4, 193.0)
- added J24: break, breakaway:0.35mil_square, B.Cu at (61.0, 193.0)
- added J25: break, breakaway:0.35mil_square, F.Cu at (58.4, 194.3)
- added J26: break, breakaway:0.35mil_square, F.Cu at (61.0, 194.3)
- added J27: break, breakaway:0.35mil_square, B.Cu at (58.4, 194.3)
- added J28: break, breakaway:0.35mil_square, B.Cu at (61.0, 194.3)
- added J29: break, breakaway:0.35mil_square, F.Cu at (72.4, 191.8)
- added J3: CONN_01X08, Pin_Headers:Pin_Header_Straight_1x08_Pitch2.54mm_SMD_Pin1Right, F.Cu at (64.1, 178.4)
- added J30: break, breakaway:0.35mil_square, F.Cu at (74.9, 191.8)
- added J31: break, breakaway:0.35mil_square, B.Cu at (72.4, 191.8)
- added J32: break, breakaway:0.35mil_square, B.Cu at (74.9, 191.8)
- added J33: break, breakaway:0.35mil_square, F.Cu at (72.4, 193.0)
- added J34: break, breakaway:0.35mil_square, F.Cu at (74.9, 193.0)
- added J35: break, breakaway:0.35mil_square, B.Cu at (72.4, 193.0)
- added J36: break, breakaway:0.35mil_square, B.Cu at (74.9, 193.0)
- added J37: break, breakaway:0.35mil_square, F.Cu at (72.4, 194.3)
- added J38: break, breakaway:0.35mil_square, F.Cu at (74.9, 194.3)
- added J39: break, breakaway:0.35mil_square, B.Cu at (72.4, 194.3)
- added J4: CONN_01X08, Pin_Headers:Pin_Header_Straight_1x08_Pitch2.54mm_SMD_Pin1Right, F.Cu at (78.1, 178.4)
- added J40: break, breakaway:0.35mil_square, B.Cu at (74.9, 194.3)
- added J41: break, breakaway:0.35mil_square, F.Cu at (86.4, 191.8)
- added J42: break, breakaway:0.35mil_square, B.Cu at (86.4, 191.8)
- added J43: break, breakaway:0.35mil_square, F.Cu at (86.4, 193.0)
- added J44: break, breakaway:0.35mil_square, B.Cu at (86.4, 193.0)
- added J45: break, breakaway:0.35mil_square, F.Cu at (86.4, 194.3)
- added J46: break, breakaway:0.35mil_square, B.Cu at (86.4, 194.3)
- added J47: CONN_01X01, SMD_Packages:1Pin, F.Cu at (20.3, 170.2)
- added J48: CONN_01X01, SMD_Packages:1Pin, F.Cu at (15.2, 175.3)
- added J49: CONN_01X01, SMD_Packages:1Pin, F.Cu at (15.2, 170.2)
- added J5: break, breakaway:0.35mil_square, F.Cu at (47.0, 191.8)
- added J6: break, breakaway:0.35mil_square, F.Cu at (44.5, 191.8)
- added J7: break, breakaway:0.35mil_square, B.Cu at (47.0, 191.8)
- added J8: break, breakaway:0.35mil_square, B.Cu at (44.5, 191.8)
- added J9: break, breakaway:0.35mil_square, F.Cu at (44.5, 193.0)
- added Mode1: TP, Measurement_Points:Measurement_Point_Round-SMD-Pad_Small, F.Cu at (22.2, 177.2)
- added Q1: A09T, TO_SOT_Packages_SMD:SOT-23, F.Cu at (34.9, 178.4)
- added Q10: A09T, TO_SOT_Packages_SMD:SOT-23, F.Cu at (53.3, 172.1)
- added Q11: A09T, TO_SOT_Packages_SMD:SOT-23, F.Cu at (55.2, 174.6)
- added Q12: A09T, TO_SOT_Packages_SMD:SOT-23, F.Cu at (53.3, 177.2)
- added Q13: A09T, TO_SOT_Packages_SMD:SOT-23, F.Cu at (55.2, 179.7)
- added Q14: A09T, TO_SOT_Packages_SMD:SOT-23, F.Cu at (53.3, 182.2)
- added Q15: A09T, TO_SOT_Packages_SMD:SOT-23, F.Cu at (55.2, 184.8)
- added Q16: A09T, TO_SOT_Packages_SMD:SOT-23, F.Cu at (53.3, 187.3)
- added Q17: A09T, TO_SOT_Packages_SMD:SOT-23, F.Cu at (69.2, 169.5)
- added Q18: A09T, TO_SOT_Packages_SMD:SOT-23, F.Cu at (67.3, 172.1)
- added Q19: A09T, TO_SOT_Packages_SMD:SOT-23, F.Cu at (69.2, 174.6)
- added Q2: A09T, TO_SOT_Packages_SMD:SOT-23, F.Cu at (34.9, 183.5)
- added Q20: A09T, TO_SOT_Packages_SMD:SOT-23, F.Cu at (67.3, 177.2)
- added Q21: A09T, TO_SOT_Packages_SMD:SOT-23, F.Cu at (69.2, 179.7)
- added Q22: A09T, TO_SOT_Packages_SMD:SOT-23, F.Cu at (67.3, 182.2)
- added Q23: A09T, TO_SOT_Packages_SMD:SOT-23, F.Cu at (69.2, 184.8)
- added Q24: A09T, TO_SOT_Packages_SMD:SOT-23, F.Cu at (67.3, 187.3)
- added Q25: A09T, TO_SOT_Packages_SMD:SOT-23, F.Cu at (83.2, 169.5)
- added Q26: A09T, TO_SOT_Packages_SMD:SOT-23, F.Cu at (81.3, 172.1)
- added Q27: A09T, TO_SOT_Packages_SMD:SOT-23, F.Cu at (83.2, 174.6)
- added Q28: A09T, TO_SOT_Packages_SMD:SOT-23, F.Cu at (81.3, 177.2)
- added Q29: A09T, TO_SOT_Packages_SMD:SOT-23, F.Cu at (83.2, 179.7)
- added Q3: A09T, TO_SOT_Packages_SMD:SOT-23, F.Cu at (37.5, 181.0)
- added Q30: A09T, TO_SOT_Packages_SMD:SOT-23, F.Cu at (81.3, 182.2)
- added Q31: A09T, TO_SOT_Packages_SMD:SOT-23, F.Cu at (83.2, 184.8)
- added Q32: A09T, TO_SOT_Packages_SMD:SOT-23, F.Cu at (81.3, 187.3)
- added Q4: A09T, TO_SOT_Packages_SMD:SOT-23, F.Cu at (37.5, 186.1)
- added Q5: A09T, TO_SOT_Packages_SMD:SOT-23, F.Cu at (40.0, 178.4)
- added Q6: A09T, TO_SOT_Packages_SMD:SOT-23, F.Cu at (40.0, 183.5)
- added Q7: A09T, TO_SOT_Packages_SMD:SOT-23, F.Cu at (42.5, 181.0)
- added Q8: A09T, TO_SOT_Packages_SMD:SOT-23, F.Cu at (42.5, 186.1)
- added Q9: A09T, TO_SOT_Packages_SMD:SOT-23, F.Cu at (55.2, 169.5)
- added R1: 1k, Resistors_SMD:R_0603_HandSoldering, F.Cu at (32.4, 193.0)
- added R2: 1k, Resistors_SMD:R_0603_HandSoldering, F.Cu at (32.4, 181.6)
- added REF**: SolderWirePad_single_0-8mmDrill, Wire_Pads:SolderWirePad_single_0-8mmDrill, F.Cu at (73.7, 194.9)
- added REF**: SolderWirePad_single_0-8mmDrill, Wire_Pads:SolderWirePad_single_0-8mmDrill, F.Cu at (45.7, 192.4)
- added REF**: SolderWirePad_single_0-8mmDrill, Wire_Pads:SolderWirePad_single_0-8mmDrill, F.Cu at (45.7, 193.7)
- added REF**: SolderWirePad_single_0-8mmDrill, Wire_Pads:SolderWirePad_single_0-8mmDrill, F.Cu at (45.7, 194.9)
- added REF**: SolderWirePad_single_0-8mmDrill, Wire_Pads:SolderWirePad_single_0-8mmDrill, F.Cu at (73.7, 191.1)
- added REF**: SolderWirePad_single_0-8mmDrill, Wire_Pads:SolderWirePad_single_0-8mmDrill, F.Cu at (73.7, 192.4)
- added REF**: SolderWirePad_single_0-8mmDrill, Wire_Pads:SolderWirePad_single_0-8mmDrill, F.Cu at (73.7, 193.7)
- added REF**: SolderWirePad_single_0-8mmDrill, Wire_Pads:SolderWirePad_single_0-8mmDrill, F.Cu at (59.7, 194.9)
- added REF**: SolderWirePad_single_0-8mmDrill, Wire_Pads:SolderWirePad_single_0-8mmDrill, F.Cu at (59.7, 191.1)
- added REF**: SolderWirePad_single_0-8mmDrill, Wire_Pads:SolderWirePad_single_0-8mmDrill, F.Cu at (59.7, 192.4)
- added REF**: SolderWirePad_single_0-8mmDrill, Wire_Pads:SolderWirePad_single_0-8mmDrill, F.Cu at (59.7, 193.7)
- added REF**: SolderWirePad_single_0-8mmDrill, Wire_Pads:SolderWirePad_single_0-8mmDrill, F.Cu at (45.7, 191.1)
- added RX1: TP, Measurement_Points:Measurement_Point_Round-SMD-Pad_Small, F.Cu at (21.0, 177.2)
- added Reset1: TP, Measurement_Points:Measurement_Point_Round-SMD-Pad_Small, F.Cu at (23.5, 177.2)
- added TX1: TP, Measurement_Points:Measurement_Point_Round-SMD-Pad_Small, F.Cu at (19.7, 177.2)
- added U1: 74HC595, Housings_SOIC:SOIC-16_3.9x9.9mm_Pitch1.27mm, F.Cu at (38.7, 193.0)
- added U2: 74HC595, Housings_SOIC:SOIC-16_3.9x9.9mm_Pitch1.27mm, F.Cu at (52.7, 193.0)
- added U3: 74HC595, Housings_SOIC:SOIC-16_3.9x9.9mm_Pitch1.27mm, F.Cu at (66.7, 193.0)
- added U4: 74HC595, Housings_SOIC:SOIC-16_3.9x9.9mm_Pitch1.27mm, F.Cu at (80.6, 193.0)
- added U5: ESP-12E, ESP8266:ESP-12E_SMD, F.Cu at (21.0, 187.3)
Routing:
- net /CLK: track 0.00 -> 101.6 mm, vias 0 -> 10
- net ADC_RCLK: track 0.00 -> 74.4 mm, vias 0 -> 9
- net Net-(R1-Pad1): track 0.00 -> 45.4 mm, vias 0 -> 3
- net /MOSI: track 0.00 -> 32.9 mm, vias 0 -> 2
- net Net-(Q25-Pad1): track 0.00 -> 32.1 mm, vias 0 -> 2
- net Net-(Q17-Pad1): track 0.00 -> 32.1 mm, vias 0 -> 2
- net Net-(Q9-Pad1): track 0.00 -> 32.1 mm, vias 0 -> 2
- net /MISO: track 0.00 -> 29.9 mm, vias 0 -> 2
- net Net-(Q27-Pad1): track 0.00 -> 27.8 mm, vias 0 -> 2
- net Net-(Q19-Pad1): track 0.00 -> 27.8 mm, vias 0 -> 2
- net Net-(Q11-Pad1): track 0.00 -> 27.8 mm, vias 0 -> 2
- net Net-(Q18-Pad1): track 0.00 -> 27.3 mm, vias 0 -> 2
- net Net-(Q10-Pad1): track 0.00 -> 27.3 mm, vias 0 -> 2
- net Net-(Q26-Pad1): track 0.00 -> 27.3 mm, vias 0 -> 2
- net Net-(Q29-Pad1): track 0.00 -> 22.6 mm, vias 0 -> 2
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- added copper zone on B.Cu, net GND
- added copper zone on F.Cu, net VCC
Other:
- board outline added: 74.3 x 29.2 mm
- net class Default: clearance 0.2 -> 0.1524; trace_width 0.25 -> 0.2032; via_dia 0.6 -> 0.6858; via_drill 0.4 -> 0.3302
- net class Power added: clearance 0.1524, trace_width 0.762, via_dia 0.6858, via_drill 0.3302
- rule trace_clearance: 0.2 -> 0.1524
- rule trace_min: 0.2 -> 0.1524
- rule via_min_drill: 0.3 -> 0.3302
- rule via_min_size: 0.4 -> 0.6858
- board text added: "12V"
- board text added: "3V3"
- board text added: "GND"
- board text added: "Mode"
- board text added: "RX"
- board text added: "Reset"
- board text added: "TX"
- board text added: "v0.1"

Commit message: begins to further develop controller
Parts:
- removed C4, C5: 1uF, Capacitors_SMD:C_0603_HandSoldering
- removed G*** (x7): LOGO, LOGO
- removed GND1, Mode1, RX1, Reset1, TX1: TP, Measurement_Points:Measurement_Point_Round-SMD-Pad_Small
- removed J10, J11, J12, J13, J14, J15, J16, J17, J18, J19, J20, J21, J22, J23, J24, J25, J26, J27, J28, J29, J30, J31, J32, J33, J34, J35, J36, J37, J38, J39, J40, J41, J42, J43, J44, J45, J46, J6, J7, J8, J9: break, breakaway:0.35mil_square
- removed J47, J48, J49: CONN_01X01, SMD_Packages:1Pin
- removed Q17, Q18, Q19, Q20, Q21, Q22, Q23, Q24, Q25, Q26, Q27, Q28, Q29, Q30, Q31, Q32: A09T, TO_SOT_Packages_SMD:SOT-23
- removed REF** (x12): SolderWirePad_single_0-8mmDrill, Wire_Pads:SolderWirePad_single_0-8mmDrill
- removed U4: 74HC595, Housings_SOIC:SOIC-16_3.9x9.9mm_Pitch1.27mm
- removed U5: ESP-12E, ESP8266:ESP-12E_SMD
- added D1: LED, LEDs:LED_0603, F.Cu at (104.8, 90.2)
- added D10: LED, LEDs:LED_0603, F.Cu at (128.9, 74.3)
- added D11: LED, LEDs:LED_0603, F.Cu at (128.9, 79.4)
- added D12: LED, LEDs:LED_0603, F.Cu at (128.9, 81.3)
- added D13: LED, LEDs:LED_0603, F.Cu at (128.9, 83.2)
- added D14: LED, LEDs:LED_0603, F.Cu at (128.9, 85.1)
- added D15: LED, LEDs:LED_0603, F.Cu at (128.9, 90.2)
- added D16: LED, LEDs:LED_0603, F.Cu at (128.9, 92.1)
- added D2: LED, LEDs:LED_0603, F.Cu at (106.0, 90.2)
- added D3: LED, LEDs:LED_0603, F.Cu at (107.3, 90.2)
- added D4: LED, LEDs:LED_0603, F.Cu at (108.6, 90.2)
- added D5: LED, LEDs:LED_0603, F.Cu at (109.9, 90.2)
- added D6: LED, LEDs:LED_0603, F.Cu at (111.1, 90.2)
- added D7: LED, LEDs:LED_0603, F.Cu at (112.4, 90.2)
- added D8: LED, LEDs:LED_0603, F.Cu at (113.7, 90.2)
- added D9: LED, LEDs:LED_0603, F.Cu at (128.9, 72.4)
- added R3: 1k, Resistors_SMD:R_0603_HandSoldering, F.Cu at (63.6, 17.3)
- added R4: 1k, Resistors_SMD:R_0603_HandSoldering, F.Cu at (55.0, 25.9)
- added RN1: R_Pack04, Resistors_SMD:R_Array_Convex_4x0603, F.Cu at (92.7, 95.2)
- added RN2: R_Pack04, Resistors_SMD:R_Array_Convex_4x0603, F.Cu at (95.9, 95.2)
- added RN3: R_Pack04, Resistors_SMD:R_Array_Convex_4x0603, F.Cu at (128.9, 76.8)
- added RN4: R_Pack04, Resistors_SMD:R_Array_Convex_4x0603, F.Cu at (128.9, 87.6)
- added TP1: GND, Measurement_Points:Measurement_Point_Round-SMD-Pad_Small, F.Cu at (51.1, 26.4)
- added TP2: TX, Measurement_Points:Measurement_Point_Round-SMD-Pad_Small, F.Cu at (59.9, 17.8)
- added TP3: RX, Measurement_Points:Measurement_Point_Round-SMD-Pad_Small, F.Cu at (67.6, 10.3)
- added TP4: MODE, Measurement_Points:Measurement_Point_Round-SMD-Pad_Small, F.Cu at (41.5, 35.2)
- added TP5: RST, Measurement_Points:Measurement_Point_Round-SMD-Pad_Small, F.Cu at (21.9, 39.6)
- J1: value CONN_02X08 -> CONN_01X01; footprint Pin_Headers:Pin_Header_Straight_2x08_Pitch2.54mm_SMD -> SMD_Packages:1Pin
- J2, J3: value CONN_01X08 -> CONN_01X01; footprint Pin_Headers:Pin_Header_Straight_1x08_Pitch2.54mm_SMD_Pin1Right -> SMD_Packages:1Pin
- J4: value CONN_01X08 -> CONN_02X08; footprint Pin_Headers:Pin_Header_Straight_1x08_Pitch2.54mm_SMD_Pin1Right -> Connectors:IDC_Header_SMD_16pins
- J5: value break -> CONN_01X08; footprint breakaway:0.35mil_square -> Pin_Headers:Pin_Header_Straight_1x08_Pitch2.54mm_SMD_Pin1Right
- U1: value 74HC595 -> ESP-12E; footprint Housings_SOIC:SOIC-16_3.9x9.9mm_Pitch1.27mm -> ESP8266:ESP-12E_SMD
- moved J2 173.6 mm to (49.5, 4.81)
- moved C1 161.9 mm to (63.3, 30.3), turned to 0 degrees
- moved R2 160.3 mm to (69.1, 25.6), turned to 0 degrees
- moved C2 158.7 mm to (67.3, 30.3), turned to 0 degrees
- moved R1 153.9 mm to (54.3, 40.7), turned to 0 degrees
- moved J1 153.5 mm to (41.7, 18.8), turned to 0 degrees
- moved J3 153.3 mm to (29.1, 29.2)
- moved C3 151.2 mm to (58.4, 37.9), turned to 0 degrees
- moved J5 131.7 mm to (120.7, 82.5)
- moved Q8 123.1 mm to (113.0, 85.1), turned to 270 degrees
- moved Q4 120.3 mm to (102.9, 85.1), turned to 270 degrees
- moved Q6 119.6 mm to (108.0, 85.1), turned to 270 degrees
- moved Q13 119.0 mm to (125.7, 83.8)
- moved Q10 119.0 mm to (123.8, 76.2)
- moved Q11 119.0 mm to (125.7, 78.7)
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Connections:
- C1 pad 1: GND -> VCC
- C1 pad 2: VCC -> GND
- C2 pad 1: GND -> VCC
- C2 pad 2: VCC -> GND
- C3 pad 1: GND -> VCC
- C3 pad 2: VCC -> GND
- J2 pad 1: N_ADC0 -> VCC
- J3 pad 1: N_ADC8 -> GND
- J4 pad 1: N_ADC16 -> +12V
- J4 pad 2: N_ADC17 -> +12V
- J4 pad 3: N_ADC18 -> GND
- J4 pad 4: N_ADC19 -> GND
- J4 pad 5: N_ADC20 -> VCC
- J4 pad 6: N_ADC21 -> /HSPI_MISO
- J4 pad 7: N_ADC22 -> /HSPI_SCK
- J4 pad 8: N_ADC23 -> N_LOAD
- J5 pad 1: VCC -> N_ADC0
- Q1 pad 1: Net-(Q1-Pad1) -> Net-(D1-Pad2)
- Q10 pad 1: Net-(Q10-Pad1) -> Net-(D10-Pad2)
- Q11 pad 1: Net-(Q11-Pad1) -> Net-(D11-Pad2)
- Q12 pad 1: Net-(Q12-Pad1) -> Net-(D12-Pad2)
- Q13 pad 1: Net-(Q13-Pad1) -> Net-(D13-Pad2)
- Q14 pad 1: Net-(Q14-Pad1) -> Net-(D14-Pad2)
- Q15 pad 1: Net-(Q15-Pad1) -> Net-(D15-Pad2)
- Q16 pad 1: Net-(Q16-Pad1) -> Net-(D16-Pad2)
- Q2 pad 1: Net-(Q2-Pad1) -> Net-(D2-Pad2)
- Q3 pad 1: Net-(Q3-Pad1) -> Net-(D3-Pad2)
- Q4 pad 1: Net-(Q4-Pad1) -> Net-(D4-Pad2)
- Q5 pad 1: Net-(Q5-Pad1) -> Net-(D5-Pad2)
- Q6 pad 1: Net-(Q6-Pad1) -> Net-(D6-Pad2)
- Q7 pad 1: Net-(Q7-Pad1) -> Net-(D7-Pad2)
- Q8 pad 1: Net-(Q8-Pad1) -> Net-(D8-Pad2)
- Q9 pad 1: Net-(Q9-Pad1) -> Net-(D9-Pad2)
- R1 pad 1: Net-(R1-Pad1) -> RST
- R2 pad 1: Net-(Mode1-Pad1) -> Net-(R2-Pad1)
- U1 pad 1: Net-(Q2-Pad1) -> RST
- U1 pad 10: VCC -> START_RCLK
- U1 pad 11: /CLK -> (no net)
- U1 pad 12: START_RCLK -> MODE
- U1 pad 13: GND -> ADC_RCLK
- U1 pad 14: /MOSI -> N_LOAD
- U1 pad 15: Net-(Q1-Pad1) -> RX
- U1 pad 16: VCC -> TX
- U1 pad 2: Net-(Q3-Pad1) -> (no net)
- U1 pad 3: Net-(Q4-Pad1) -> Net-(R2-Pad1)
- U1 pad 4: Net-(Q5-Pad1) -> (no net)
- U1 pad 5: Net-(Q6-Pad1) -> /HSPI_SCK
- U1 pad 6: Net-(Q7-Pad1) -> /HSPI_MISO
- U1 pad 7: Net-(Q8-Pad1) -> /HSPI_MOSI
- U1 pad 8: GND -> VCC
- U1 pad 9: (no net) -> GND
- U2 pad 1: Net-(Q10-Pad1) -> Net-(D2-Pad2)
- U2 pad 11: /CLK -> /HSPI_SCK
- U2 pad 12: ADC_RCLK -> START_RCLK
- U2 pad 14: /MOSI -> /HSPI_MOSI
- U2 pad 15: Net-(Q9-Pad1) -> Net-(D1-Pad2)
- U2 pad 2: Net-(Q11-Pad1) -> Net-(D3-Pad2)
- U2 pad 3: Net-(Q12-Pad1) -> Net-(D4-Pad2)
- U2 pad 4: Net-(Q13-Pad1) -> Net-(D5-Pad2)
- U2 pad 5: Net-(Q14-Pad1) -> Net-(D6-Pad2)
- U2 pad 6: Net-(Q15-Pad1) -> Net-(D7-Pad2)
- U2 pad 7: Net-(Q16-Pad1) -> Net-(D8-Pad2)
- U2 pad 9: Net-(J21-Pad1) -> (no net)
- U3 pad 1: Net-(Q18-Pad1) -> Net-(D10-Pad2)
- U3 pad 11: /CLK -> /HSPI_SCK
- U3 pad 14: Net-(J21-Pad1) -> /HSPI_MOSI
- U3 pad 15: Net-(Q17-Pad1) -> Net-(D9-Pad2)
- U3 pad 2: Net-(Q19-Pad1) -> Net-(D11-Pad2)
- U3 pad 3: Net-(Q20-Pad1) -> Net-(D12-Pad2)
- U3 pad 4: Net-(Q21-Pad1) -> Net-(D13-Pad2)
- U3 pad 5: Net-(Q22-Pad1) -> Net-(D14-Pad2)
- U3 pad 6: Net-(Q23-Pad1) -> Net-(D15-Pad2)
- U3 pad 7: Net-(Q24-Pad1) -> Net-(D16-Pad2)
- U3 pad 9: Net-(J33-Pad1) -> (no net)
Routing:
- net /CLK: track 101.6 -> 0.00 mm, vias 10 -> 0
- net ADC_RCLK: track 74.4 -> 0.00 mm, vias 9 -> 0
- net Net-(R1-Pad1): track 45.4 -> 0.00 mm, vias 3 -> 0
- net Net-(D10-Pad2): track 0.00 -> 34.7 mm, vias 0 -> 2
- net Net-(D9-Pad2): track 0.00 -> 33.1 mm, vias 0 -> 3
- net /MOSI: track 32.9 -> 0.00 mm, vias 2 -> 0
- net Net-(Q25-Pad1): track 32.1 -> 0.00 mm, vias 2 -> 0
- net Net-(Q17-Pad1): track 32.1 -> 0.00 mm, vias 2 -> 0
- net Net-(Q9-Pad1): track 32.1 -> 0.00 mm, vias 2 -> 0
- net /MISO: track 29.9 -> 0.00 mm, vias 2 -> 0
- net Net-(D11-Pad2): track 0.00 -> 29.3 mm, vias 0 -> 2
- net Net-(D12-Pad2): track 0.00 -> 28.9 mm, vias 0 -> 2
- net Net-(Q27-Pad1): track 27.8 -> 0.00 mm, vias 2 -> 0
- net Net-(Q19-Pad1): track 27.8 -> 0.00 mm, vias 2 -> 0
- net Net-(Q11-Pad1): track 27.8 -> 0.00 mm, vias 2 -> 0
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Other:
- board size 74.3 x 29.2 mm -> 80.6 x 29.2 mm
- board text removed: "12V"
- board text removed: "3V3"
- board text removed: "GND"
- board text removed: "Mode"
- board text removed: "RX"
- board text removed: "Reset"
- board text removed: "TX"
- board text removed: "v0.1"
